File: PCB/Button/mai_button.kicad_sch (KiCad schematic)
At the start: 14 parts, among them J1 Conn_01x03, J2 Conn_01x02, J3 Conn_01x03, J4 Conn_01x02, SW1 SW_DIP_x01

Commit message: Button PCB update (v1.1)
Parts:
- removed J2, J4: Conn_01x02, mai_button:Solder_2P, symbol Connector_Generic:Conn_01x02
- added J2, J4: Btn, mai_button:Solder_1P, symbol Connector_Generic:Conn_01x01
- J1: value Conn_01x03 -> RGB In
- J3: value Conn_01x03 -> RGB Out
Connections:
- net GND: now also SW1.1
- net at SW1.2: now also J2.1 (Pin_1), J4.1 (Pin_1)
