File: PCB/IO/mai_io.kicad_pcb (KiCad board)
At the start: 2 copper layers, 98 x 80 mm, 43 parts, among them J1 Conn_01x34_Female, U1 Pico, U2 MPR121QR2, U3 MPR121QR2, U4 MPR121QR2, U5 MPR121QR2_BOARD, U6 MPR121QR2_BOARD, U7 MPR121QR2_BOARD, U8 SN74LV1T34DBV

Commit message: IO board v1.1 (better support for arcade buttons and simplified)
Parts:
- removed the C1 at (77.8, 71.2)
- removed C10, C2, C4, C5, C6, C7, C8, C9: 0.1uF, Capacitor_SMD:C_0603_1608Metric_Pad1.08x0.95mm_HandSolder
- removed U2, U3, U4: MPR121QR2, Package_DFN_QFN:UQFN-20_3x3mm_P0.4mm
- removed U8: SN74LV1T34DBV, mai_io:SOT-23-5_Jumper
- added R10: 10K, Resistor_SMD:R_0603_1608Metric_Pad0.98x0.95mm_HandSolder, B.Cu at (94.7, 82.1)
- added R11: 10K, Resistor_SMD:R_0603_1608Metric_Pad0.98x0.95mm_HandSolder, B.Cu at (99.8, 82.1)
- added R12: 10K, Resistor_SMD:R_0603_1608Metric_Pad0.98x0.95mm_HandSolder, B.Cu at (102.3, 82.1)
- added R13: 10K, Resistor_SMD:R_0603_1608Metric_Pad0.98x0.95mm_HandSolder, B.Cu at (104.9, 82.1)
- added R14: 10K, Resistor_SMD:R_0603_1608Metric_Pad0.98x0.95mm_HandSolder, B.Cu at (107.4, 82.1)
- added R15: 10K, Resistor_SMD:R_0603_1608Metric_Pad0.98x0.95mm_HandSolder, B.Cu at (117.6, 82.1)
- added R16: 10K, Resistor_SMD:R_0603_1608Metric_Pad0.98x0.95mm_HandSolder, B.Cu at (120.1, 82.1)
- added R5: 220, Resistor_SMD:R_0603_1608Metric_Pad0.98x0.95mm_HandSolder, B.Cu at (113.8, 98.6)
- added R6: 220, Resistor_SMD:R_0603_1608Metric_Pad0.98x0.95mm_HandSolder, B.Cu at (125.8, 98.6)
- added R7: 220, Resistor_SMD:R_0603_1608Metric_Pad0.98x0.95mm_HandSolder, B.Cu at (137.8, 98.6)
- added R8: 220, Resistor_SMD:R_0603_1608Metric_Pad0.98x0.95mm_HandSolder, B.Cu at (149.8, 98.6)
- added R9: 10K, Resistor_SMD:R_0603_1608Metric_Pad0.98x0.95mm_HandSolder, B.Cu at (92.2, 82.1)
- R1, R2, R3: value 75K -> 220; footprint Resistor_SMD:R_0603_1608Metric -> Resistor_SMD:R_0603_1608Metric_Pad0.98x0.95mm_HandSolder; moved to B.Cu
- R20, R21: footprint Resistor_SMD:R_0603_1608Metric -> Resistor_SMD:R_0603_1608Metric_Pad0.98x0.95mm_HandSolder
- R4: value 10 -> 220; footprint Resistor_SMD:R_0603_1608Metric -> Resistor_SMD:R_0603_1608Metric_Pad0.98x0.95mm_HandSolder; moved to B.Cu
- U1: value Pico -> PiPico
- moved R4 52.1 mm to (101.8, 98.6), turned to -90 degrees
- moved R3 46.0 mm to (89.8, 98.6), turned to -90 degrees
- moved R2 27.2 mm to (77.8, 98.6), turned to -90 degrees
- moved R1 12.7 mm to (65.8, 98.6), turned to -90 degrees
- moved R20 2.00 mm to (83.6, 73.2)
- moved R21 2.00 mm to (80.6, 73.2)
- renumbered C3 to C1
Connections:
- BT1 pad 1: +5V -> Net-(BT1-Pin_1)
- BT2 pad 1: +5V -> Net-(BT2-Pin_1)
- BT3 pad 1: +5V -> Net-(BT3-Pin_1)
- BT4 pad 1: +5V -> Net-(BT4-Pin_1)
- BT5 pad 1: +5V -> Net-(BT5-Pin_1)
- BT6 pad 1: +5V -> Net-(BT6-Pin_1)
- BT7 pad 1: +5V -> Net-(BT7-Pin_1)
- BT8 pad 1: +5V -> Net-(BT8-Pin_1)
- R1 pad 1: Net-(R1-Pad1) -> Net-(BT1-Pin_1)
- R1 pad 2: GND -> +5V
- R2 pad 1: Net-(R2-Pad1) -> Net-(BT2-Pin_1)
- R2 pad 2: GND -> +5V
- R3 pad 1: Net-(R3-Pad1) -> Net-(BT3-Pin_1)
- R3 pad 2: GND -> +5V
- R4 pad 1: Net-(R4-Pad1) -> Net-(BT4-Pin_1)
- R4 pad 2: Net-(R4-Pad2) -> +5V
- RGB0 pad 2: Net-(R4-Pad1) -> Net-(RGB0-Pin_2)
- U1 pad 17: Net-(R4-Pad2) -> Net-(RGB0-Pin_2)
- U1 pad 39: unconnected-(U1-Pad39) -> +5V
- U1 pad 40: +5V -> unconnected-(U1-VBUS-Pad40)
- USB1 pad 13: unconnected-(USB1-Pad13) -> GND
Routing:
- net /SDA: track 157.3 -> 116.2 mm
- net /SCL: track 140.6 -> 108.9 mm
- net GND: track 33.0 -> 3.46 mm, vias 13 -> 27
- net Net-(RGB0-Pin_2): track 0.00 -> 27.8 mm
- net Net-(R4-Pad2): track 25.2 -> 0.00 mm
- net +3V3: track 168.0 -> 143.2 mm
- net +5V: track 253.4 -> 232.1 mm, vias 0 -> 9
- net /B12: track 34.7 -> 14.5 mm
- net unconnected-(USB1-Pad13): track 17.0 -> 0.00 mm
- net /B1: track 32.7 -> 16.2 mm
- net /A12: track 35.8 -> 19.3 mm
- net /A1: track 45.9 -> 29.5 mm
- net /C1: track 32.1 -> 15.7 mm
- net /C12: track 16.4 -> 0.00 mm
- net /B2: track 31.4 -> 15.4 mm
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Other:
- board text added: "Mai Pico v1.1"
- board text removed: "Mai Pico v1.0"
